Commit message: added needle

File: ur_description/urdf/inc/ur_common.xacro (robot description, xacro)
@@ -189,4 +189,16 @@
     <xacro:property name="wrist_3_collision_mesh" value="${wrist_3_mesh['collision']['mesh']}" scope="parent"/>
     <xacro:property name="wrist_3_visual_offset" value="${wrist_3_mesh['visual_offset']}" scope="parent"/>
+    <xacro:property name="holder_mesh" value="${sec_mesh_files['holder']}"/>
+    <xacro:property name="holder_visual_mesh" value="${holder_mesh['visual']['mesh']}" scope="parent"/>
+    <xacro:property name="holder_collision_mesh" value="${holder_mesh['collision']['mesh']}" scope="parent"/>
+    <xacro:property name="holder_visual_offset" value="${holder_mesh['visual_offset']}" scope="parent"/>
+    <xacro:property name="holder_visual_material_name" value="${holder_mesh['visual']['material']['name']}" scope="parent"/>
+    <xacro:property name="holder_visual_material_color" value="${holder_mesh['visual']['material']['color']}" scope="parent"/>
+    <xacro:property name="needle_mesh" value="${sec_mesh_files['needle']}"/>
+    <xacro:property name="needle_visual_mesh" value="${needle_mesh['visual']['mesh']}" scope="parent"/>
+    <xacro:property name="needle_collision_mesh" value="${needle_mesh['collision']['mesh']}" scope="parent"/>
+    <xacro:property name="needle_visual_offset" value="${needle_mesh['visual_offset']}" scope="parent"/>
+    <xacro:property name="needle_visual_material_name" value="${needle_mesh['visual']['material']['name']}" scope="parent"/>
+    <xacro:property name="needle_visual_material_color" value="${needle_mesh['visual']['material']['color']}" scope="parent"/>
     <!--KINEMATICS HASH-->
     <xacro:property name="kinematics_hash" value="${sec_kinematics['hash']}" scope="parent"/>

File: ur_description/urdf/ur_macro.xacro (robot description, xacro)
@@ -329,4 +329,51 @@
       <origin xyz="0 0 0" rpy="0 ${-pi/2.0} ${-pi/2.0}" />
     </joint>
+    <link name="${prefix}holder">
+      <visual>
+        <origin xyz="0 0 0" rpy="0 0 0"/>
+        <geometry>
+          <mesh filename="${holder_visual_mesh}"/>
+        </geometry>
+        <material name="${holder_visual_material_name}">
+          <color rgba="${holder_visual_material_color}"/>
+        </material>
+      </visual>
+      <collision>
+        <origin xyz="0 0 ${holder_visual_offset}" rpy="0 0 0"/>
+        <geometry>
+          <mesh filename="${holder_collision_mesh}"/>
+        </geometry>
+      </collision>
+    </link>
+    <joint name="${prefix}wrist_3-holder" type="fixed">
+        <parent link="${prefix}wrist_3_link" />
+        <child link="${prefix}holder" />
+        <origin xyz="0 0 0" rpy="0 ${-pi} 0" />
+    </joint>
+    <link name="${prefix}needle">
+      <visual>
+        <origin xyz="0 0 0" rpy="0 0 0"/>
+        <geometry>
+          <mesh filename="${needle_visual_mesh}"/>
+        </geometry>
+        <material name="${needle_visual_material_name}">
+          <color rgba="${needle_visual_material_color}"/>
+        </material>
+      </visual>
+      <collision>
+        <origin xyz="0 0 ${needle_visual_offset}" rpy="0 0 0"/>
+        <geometry>
+          <mesh filename="${needle_collision_mesh}"/>
+        </geometry>
+      </collision>
+    </link>
+    <joint name="${prefix}holder-needle" type="prismatic">
+        <parent link="${prefix}holder" />
+        <child link="${prefix}needle" />
+        <origin xyz="0 0 -0.1475" rpy="${-pi/2.0} 0 0" />
+        <axis xyz="0 0 1" />
+        <limit lower="0" upper="0.1"
+               effort="-5" velocity="0.01"/>
+    </joint>
     <!-- ROS-Industrial 'tool0' frame - all-zeros tool frame -->
     <link name="${prefix}tool0"/>

File: ur_moveit_config/srdf/ur_macro.srdf.xacro (robot description, xacro)
@@ -54,4 +54,6 @@
     <disable_collisions link1="${prefix}wrist_1_link" link2="${prefix}wrist_3_link" reason="Never" />
     <disable_collisions link1="${prefix}wrist_2_link" link2="${prefix}wrist_3_link" reason="Adjacent" />
+    <disable_collisions link1="${prefix}wrist_3_link" link2="${prefix}holder" reason="Adjacent" />
+    <disable_collisions link1="${prefix}holder" link2="${prefix}needle" reason="Adjacent" />
   </xacro:macro>
 </robot>
