Commit message: scene update and kinematics

File: ur_description/urdf/ur_macro.xacro (robot description, xacro)
@@ -349,5 +349,5 @@
         <parent link="${prefix}wrist_3_link" />
         <child link="${prefix}holder" />
-        <origin xyz="0 0 0" rpy="0 ${-pi} 0" />
+        <origin xyz="0 0 0" rpy="0 ${-pi} 2.356194490192345" />
     </joint>
     <link name="${prefix}needle">
@@ -368,11 +368,15 @@
       </collision>
     </link>
-    <joint name="${prefix}holder-needle" type="prismatic">
+    <joint name="${prefix}holder-needle" type="fixed">
         <parent link="${prefix}holder" />
         <child link="${prefix}needle" />
-        <origin xyz="0 0 -0.1475" rpy="${-pi/2.0} 0 0" />
-        <axis xyz="0 0 1" />
-        <limit lower="0" upper="0.1"
-               effort="-5" velocity="0.01"/>
+        <origin xyz="0 0.092 -0.1475" rpy="${-pi/2.0} 0 0" />
+    </joint>
+    <link name="${prefix}tip">
+    </link>
+    <joint name="${prefix}needle-tip" type="fixed">
+        <parent link="${prefix}needle" />
+        <child link="${prefix}tip" />
+        <origin xyz="0 0 0.025" rpy="0 0 0" />
     </joint>
     <!-- ROS-Industrial 'tool0' frame - all-zeros tool frame -->
